File: PCB/Instruments/Instruments/Instruments.kicad_sch (KiCad schematic)
At the start: 8 parts, among them P1 Screw-Terminal-1x2, U1 SEEEDUINO XIAO, U2 LD33VT

Commit message: Finished Code + PCB
Parts:
- removed C2: 10uF, Instruments:100UFX16V CAPACITOR D5.0XF11.0, symbol 100UFx16V capacitor D5.0xF11.0
- removed H1: 2.54mm 1*6P, Instruments:HDR-2.54-15-1X6P, symbol 2.54mm 1*6P
- added C2: 10uF, Instruments:CAP-TH_L4.2-W3.8-P2.54-D0.5, symbol CT4-0805Y104M500
- added D1: IR204A, LED_THT:LED_D3.0mm_IRBlack, symbol LED:IR204A
- added R1: R220, Resistor_THT:R_Array_SIP4, symbol Device:R
- added U3: 7 pin JST Connector, Instruments:HDR-2.54-15-1X6P, symbol 7 pin JST Connector
- H3: value HDR-F-2.54_1x2 -> 2.54mm 1*2P
- LCD1: value SSD1306-OLED-128X64-I2C-VIZNY DEBORA -> SSD1306-OLED-128X64-I2C
Connections:
- net +3V3: now also C2.2, D1.2 (A), U3.7
- net GND: now also C2.1, R1.2, U3.6
- net LEDTCS: now also U3.1
- net SCL: now also U3.4
- net SDA: now also U3.3
- new net: D1.1 (K), R1.1
- no-connect marks 9 -> 10
